Commit message: car not moving but added maze...

File: urdf/simple_two_wheel_car.urdf (robot description, URDF)
Before this commit: robot simple_four_wheel_car, 11 links, 10 joints
Joints:
- removed joint front_wheel_joint
- added joint left_wheel_joint: type continuous, parent base_link, child left_wheel_link, origin xyz=0.0 -0.1625 -0.05 rpy=0 0 0, axis 0 1 0
