Commit message: its going in circles

File: urdf/maze.urdf (robot description, URDF)
Before this commit: robot maze, 1 links, 0 joints
Links:
- link maze_link: geometry collision box size=0.2 10 1; collision box size=0.2 10 1

Commit message: added different maze, multi envs works, trained long but doesnt find new goal

File: urdf/maze.urdf (robot description, URDF)
Before this commit: robot maze, 1 links, 0 joints
Links:
- link maze_link: geometry collision box size=0.2 2 1; collision box size=0.2 2 1
